File: AttinyProgramer/board-beta1.2v.sch (EAGLE design)
At the start: 14 parts, among them IC1 ATTINY44-SSU

Commit message: clea
Parts:
- added R6, R7: 49 Ω, fab:RES-US1206FAB
- R1, R2: value 449 Ω -> 49 Ω
Connections:
- new net N$5: R6.2, R7.1
- net D-: now also R7.2
- net GND: now also D1.ANODE, D2.ANODE; no longer D1.CATHODE, D2.CATHODE
- net VCC: now also R6.1
- net _D+: now also D1.CATHODE; no longer D1.ANODE
- net _D-: now also D2.CATHODE; no longer D2.ANODE
Other:
- note added: "Esteban Martin Gimenez"
- note added: "External VCC 5volts."
- note added: "ISP Programmer v 0.1.2"
- moved on the sheet: D1, D2
Changed lines of the file:
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@@
 <part name="D1" library="fab" deviceset="ZENER_DIODE" device="SOD123"/>
 <part name="D2" library="fab" deviceset="ZENER_DIODE" device="SOD123"/>
-<part name="R1" library="fab" deviceset="RES-US" device="1206FAB" value="449 Ω"/>
-<part name="R2" library="fab" deviceset="RES-US" device="1206FAB" value="449 Ω"/>
+<part name="R1" library="fab" deviceset="RES-US" device="1206FAB" value="49 Ω"/>
+<part name="R2" library="fab" deviceset="RES-US" device="1206FAB" value="49 Ω"/>
 <part name="SUPPLY2" library="supply2" deviceset="GND" device=""/>
 <part name="SUPPLY7" library="supply2" deviceset="GND" device=""/>
 <part name="JP1" library="pinhead" deviceset="PINHD-1X2" device=""/>
+<part name="R6" library="fab" deviceset="RES-US" device="1206FAB" value="49 Ω"/>
+<part name="R7" library="fab" deviceset="RES-US" device="1206FAB" value="49 Ω"/>
 </parts>
 <sheets>
 <sheet>
 <plain>
+<text x="129.54" y="2.54" size="1.778" layer="94" font="vector">Esteban Martin Gimenez</text>
+<text x="76.2" y="2.54" size="1.778" layer="94" font="vector">ISP Programmer v 0.1.2</text>
+<text x="-68.58" y="63.5" size="1.016" layer="94" font="vector">External VCC 5volts.</text>
 </plain>
 <instances>
@@
 <instance part="P+3" gate="VCC" x="114.3" y="106.68"/>
 <instance part="U$5" gate="G$1" x="-63.5" y="88.9" rot="R180"/>
-<instance part="D1" gate="1" x="-55.88" y="81.28" rot="R270"/>
-<instance part="D2" gate="1" x="-48.26" y="81.28" rot="R270"/>
+<instance part="D1" gate="1" x="-55.88" y="81.28" rot="R90"/>
+<instance part="D2" gate="1" x="-48.26" y="81.28" rot="R90"/>
 <instance part="R1" gate="G$1" x="-35.56" y="91.44"/>
 <instance part="R2" gate="G$1" x="-35.56" y="83.82"/>
@@
 <instance part="SUPPLY7" gate="GND" x="-48.26" y="73.66"/>
 <instance part="JP1" gate="G$1" x="-68.58" y="58.42" rot="R180"/>
+<instance part="R6" gate="G$1" x="-58.42" y="40.64"/>
+<instance part="R7" gate="G$1" x="-48.26" y="35.56" rot="R270"/>
 </instances>
 <busses>
@@
 </segment>
 <segment>
-<pinref part="D1" gate="1" pin="CATHODE"/>
-<pinref part="SUPPLY2" gate="GND" pin="GND"/>
-<wire x1="-55.88" y1="78.74" x2="-55.88" y2="76.2" width="0.1524" layer="91"/>
-</segment>
-<segment>
-<pinref part="D2" gate="1" pin="CATHODE"/>
-<pinref part="SUPPLY7" gate="GND" pin="GND"/>
-<wire x1="-48.26" y1="78.74" x2="-48.26" y2="76.2" width="0.1524" layer="91"/>
-</segment>
-<segment>
 <pinref part="JP1" gate="G$1" pin="1"/>
 <wire x1="-66.04" y1="55.88" x2="-53.34" y2="55.88" width="0.1524" layer="91"/>
 <label x="-50.8" y="53.34" size="1.778" layer="95" xref="yes"/>
+</segment>
+<segment>
+<pinref part="D1" gate="1" pin="ANODE"/>
+<pinref part="SUPPLY2" gate="GND" pin="GND"/>
+<wire x1="-55.88" y1="78.74" x2="-55.88" y2="76.2" width="0.1524" layer="91"/>
+</segment>
+<segment>
+<pinref part="D2" gate="1" pin="ANODE"/>
+<pinref part="SUPPLY7" gate="GND" pin="GND"/>
+<wire x1="-48.26" y1="78.74" x2="-48.26" y2="76.2" width="0.1524" layer="91"/>
 </segment>
 </net>
@@
 <label x="-50.8" y="60.96" size="1.778" layer="95" xref="yes"/>
 </segment>
+<segment>
+<pinref part="R6" gate="G$1" pin="1"/>
+<wire x1="-63.5" y1="40.64" x2="-68.58" y2="40.64" width="0.1524" layer="91"/>
+<label x="-76.2" y="40.64" size="1.778" layer="95"/>
+</segment>
 </net>
 <net name="N$1" class="0">
@@
 <label x="-22.86" y="91.44" size="1.778" layer="95" xref="yes"/>
 </segment>
+<segment>
+<pinref part="R7" gate="G$1" pin="2"/>
+<wire x1="-48.26" y1="30.48" x2="-48.26" y2="25.4" width="0.1524" layer="91"/>
+<label x="-45.72" y="25.4" size="1.778" layer="95"/>
+</segment>
 </net>
 <net name="D+" class="0">
@@
 <wire x1="-55.88" y1="86.36" x2="-43.18" y2="86.36" width="0.1524" layer="91"/>
 <wire x1="-43.18" y1="86.36" x2="-40.64" y2="83.82" width="0.1524" layer="91"/>
-<pinref part="D1" gate="1" pin="ANODE"/>
+<pinref part="D1" gate="1" pin="CATHODE"/>
 <wire x1="-55.88" y1="83.82" x2="-55.88" y2="86.36" width="0.1524" layer="91"/>
 <junction x="-55.88" y="86.36"/>
@@
 <pinref part="R1" gate="G$1" pin="1"/>
 <wire x1="-60.96" y1="88.9" x2="-48.26" y2="88.9" width="0.1524" layer="91"/>
-<pinref part="D2" gate="1" pin="ANODE"/>
 <wire x1="-48.26" y1="88.9" x2="-43.18" y2="88.9" width="0.1524" layer="91"/>
 <wire x1="-43.18" y1="88.9" x2="-40.64" y2="91.44" width="0.1524" layer="91"/>
+<pinref part="D2" gate="1" pin="CATHODE"/>
 <wire x1="-48.26" y1="83.82" x2="-48.26" y2="88.9" width="0.1524" layer="91"/>
 <junction x="-48.26" y="88.9"/>
 </segment>
 </net>
+<net name="N$5" class="0">
+<segment>
+<pinref part="R6" gate="G$1" pin="2"/>
+<pinref part="R7" gate="G$1" pin="1"/>
+<wire x1="-53.34" y1="40.64" x2="-48.26" y2="40.64" width="0.1524" layer="91"/>
+</segment>
+</net>
