File: AttinyProgramer/board-beta2.0v.brd (EAGLE design)
At the start: 37.1 x 39.7 mm, 14 parts, among them IC1 ATTINY44-SSU

Commit message: clea
Parts:
- added R6, R7: 49 Ω, fab:R1206FAB
- R1, R2: value 449 Ω -> 49 Ω
- moved JP1 0.12 mm to (21.6, 34.8)
Connections:
- new net N$5: R6.2, R7.1
- net D-: now also R7.2
- net GND: now also D1.ANODE, D2.ANODE; no longer D1.CATHODE, D2.CATHODE
- net VCC: now also R6.1
- net _D+: now also D1.CATHODE; no longer D1.ANODE
- net _D-: now also D2.CATHODE; no longer D2.ANODE
Routing:
- net _D+: track 6.25 -> 14.6 mm
- net VCC: track 99.5 -> 105.6 mm
- net _D-: track 5.97 -> 10.7 mm
- net N$5: track 0.00 -> 3.26 mm
- net GND: track 75.7 -> 73.3 mm
- net D-: track 12.8 -> 13.9 mm
- net SCK: track 47.1 -> 47.7 mm
Other:
- board size 37.1 x 39.7 mm -> 37.1 x 42.7 mm
- board text added: "Boot"
- board text added: "VCC"
- board text removed: "Bootloader"
